File: esp32-pcb/esp32-pcb.kicad_pcb (KiCad board)
At the start: 2 copper layers, 35 parts, among them Q1 SS8050-G, Q2 SS8050-G, U1 CP2102N-A02-GQFN28, U2 BQ24075RGTR, U3 AP2112K-3.3TRG1, X1 ESP32-S3-WROOM-1-N16R8, Y1 Crystal

Commit message: updates
Parts:
- added J3: Conn_01x19, Connector_PinHeader_2.54mm:PinHeader_1x19_P2.54mm_Vertical, F.Cu at (127.3, 84.7)
- added J4: Conn_01x19, Connector_PinHeader_2.54mm:PinHeader_1x19_P2.54mm_Vertical, F.Cu at (150.1, 84.7)
- moved R4 33.0 mm to (98.7, 58.1)
- moved C1 33.0 mm to (114.7, 64.8)
- moved C2 33.0 mm to (119.6, 66.4)
- moved C3 33.0 mm to (101.6, 59.2)
- moved C5 33.0 mm to (101.6, 62.5)
- moved C6 33.0 mm to (101.6, 64.1)
- moved C7 33.0 mm to (101.6, 65.8)
- moved Q1 33.0 mm to (102.5, 56.1)
- moved Q2 33.0 mm to (106.9, 56.1)
- moved R1 33.0 mm to (117.0, 61.0)
- moved R2 33.0 mm to (98.7, 54.2)
- moved R3 33.0 mm to (98.7, 56.1)
- moved R5 33.0 mm to (98.7, 60.1)
- moved R7 33.0 mm to (98.7, 64.1)
- moved R8 33.0 mm to (98.7, 66.1)
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
Commit message: updates
Parts:
- added D2: LED, Diode_SMD:D_0603_1608Metric_Pad1.05x0.95mm_HandSolder, F.Cu at (81.7, 72.3)
- added D3: LED, Diode_SMD:D_0603_1608Metric_Pad1.05x0.95mm_HandSolder, F.Cu at (81.7, 74.9)
- added J1: USB_B_Micro, USB-micro-receptacle:CUI_UJ2-MIBH2-4-SMT, F.Cu at (142.4, 128.2)
- added J2: USB_B_Micro, USB-micro-receptacle:CUI_UJ2-MIBH2-4-SMT, F.Cu at (133.2, 128.2)
- added J5: Batt+, Connector_PinHeader_2.54mm:PinHeader_1x01_P2.54mm_Vertical, F.Cu at (127.5, 125.0)
- added J6: Batt-, Connector_PinHeader_2.54mm:PinHeader_1x01_P2.54mm_Vertical, F.Cu at (127.5, 129.8)
- C1, C10, C11, C12, C2, C3, C4, C5, C6, C7, C8, C9: footprint Capacitor_SMD:C_01005_0402Metric_Pad0.57x0.30mm_HandSolder -> Capacitor_SMD:C_0402_1005Metric_Pad0.74x0.62mm_HandSolder
- J3: value Conn_01x19 -> Conn_01x15; footprint Connector_PinHeader_2.54mm:PinHeader_1x19_P2.54mm_Vertical -> Connector_PinHeader_2.54mm:PinHeader_1x15_P2.54mm_Vertical
- moved R3 77.2 mm to (147.5, 116.0), turned to 90 degrees
- moved R4 74.9 mm to (146.2, 116.0), turned to 90 degrees
- moved R5 72.6 mm to (145.0, 116.0), turned to -90 degrees
- moved R6 69.4 mm to (142.5, 116.0), turned to -90 degrees
- moved C6 66.8 mm to (143.8, 116.0), turned to -90 degrees
- moved C7 64.0 mm to (141.2, 116.0), turned to 90 degrees
- moved Q1 61.0 mm to (139.0, 105.0), turned to 90 degrees
- moved R2 60.7 mm to (130.8, 105.8), turned to 180 degrees
- moved Q2 60.7 mm to (142.9, 105.0), turned to 90 degrees
- moved C3 59.2 mm to (130.8, 110.8), turned to 180 degrees
- moved R11 59.1 mm to (130.8, 117.0)
- moved U2 58.9 mm to (135.4, 114.5), turned to 90 degrees
- moved C4 58.9 mm to (130.8, 112.0), turned to 180 degrees
- moved R8 58.8 mm to (140.5, 107.5), turned to 180 degrees
- moved R9 58.7 mm to (139.2, 111.2)
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Connections:
- J3 pad 1: unconnected-(J3-Pin_1-Pad1) -> /VDD_ESP
- J3 pad 10: unconnected-(J3-Pin_10-Pad10) -> /IO8
- J3 pad 11: unconnected-(J3-Pin_11-Pad11) -> /IO3
- J3 pad 12: unconnected-(J3-Pin_12-Pad12) -> GND
- J3 pad 13: unconnected-(J3-Pin_13-Pad13) -> GND
- J3 pad 14: unconnected-(J3-Pin_14-Pad14) -> /VDD_SYS
- J3 pad 15: unconnected-(J3-Pin_15-Pad15) -> /VDD_SYS
- J3 pad 2: unconnected-(J3-Pin_2-Pad2) -> /VDD_ESP
- J3 pad 3: unconnected-(J3-Pin_3-Pad3) -> /CHIP_PU
- J3 pad 4: unconnected-(J3-Pin_4-Pad4) -> /IO4
- J3 pad 5: unconnected-(J3-Pin_5-Pad5) -> /IO5
- J3 pad 6: unconnected-(J3-Pin_6-Pad6) -> /IO6
- J3 pad 7: unconnected-(J3-Pin_7-Pad7) -> /IO7
- J3 pad 8: unconnected-(J3-Pin_8-Pad8) -> /IO17
- J3 pad 9: unconnected-(J3-Pin_9-Pad9) -> /IO18
- J4 pad 1: unconnected-(J4-Pin_1-Pad1) -> /VDD_ESP
- J4 pad 10: unconnected-(J4-Pin_10-Pad10) -> /IO38
- J4 pad 11: unconnected-(J4-Pin_11-Pad11) -> /IO37
- J4 pad 12: unconnected-(J4-Pin_12-Pad12) -> /IO36
- J4 pad 13: unconnected-(J4-Pin_13-Pad13) -> /IO35
- J4 pad 14: unconnected-(J4-Pin_14-Pad14) -> /IO0
- J4 pad 2: unconnected-(J4-Pin_2-Pad2) -> /IO1
- J4 pad 3: unconnected-(J4-Pin_3-Pad3) -> /IO2
- J4 pad 4: unconnected-(J4-Pin_4-Pad4) -> /CP_RXD
- J4 pad 5: unconnected-(J4-Pin_5-Pad5) -> /CP_TXD
- J4 pad 6: unconnected-(J4-Pin_6-Pad6) -> /IO42
- J4 pad 7: unconnected-(J4-Pin_7-Pad7) -> /IO41
- J4 pad 8: unconnected-(J4-Pin_8-Pad8) -> /IO40
- J4 pad 9: unconnected-(J4-Pin_9-Pad9) -> /IO39
Routing:
- net /VDD_USB: track 0.00 -> 42.2 mm, vias 0 -> 3
- net /CHIP_PU: track 0.00 -> 35.8 mm, vias 0 -> 2
- net /D-: track 0.00 -> 32.4 mm
- net /VDD_SYS: track 0.00 -> 31.1 mm, vias 0 -> 5
- net /D+: track 0.00 -> 30.7 mm
- net /CP_TXD: track 0.00 -> 29.9 mm, vias 0 -> 2
- net /CP_RXD: track 0.00 -> 29.0 mm, vias 0 -> 3
- net Net-(X1-IO15): track 0.00 -> 27.3 mm, vias 0 -> 2
- net /IO0: track 0.00 -> 24.4 mm
- net Net-(X1-IO16): track 0.00 -> 23.2 mm, vias 0 -> 2
- net /USB_D+: track 0.00 -> 20.1 mm, vias 0 -> 2
- net /IO35: track 0.00 -> 18.9 mm, vias 0 -> 1
- net /USB_D-: track 0.00 -> 18.9 mm, vias 0 -> 2
- net /VDD_ESP: track 0.00 -> 18.1 mm, vias 0 -> 4
- net /IO36: track 0.00 -> 17.1 mm, vias 0 -> 1
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- added copper zone on B.Cu, net /VDD_SYS
- added copper zone on F.Cu, net /VDD_SYS
Other:
- board outline added: 27.5 x 51 mm

Commit message: updates from work
Connections:
- J4 pad 15: unconnected-(J4-Pin_15-Pad15) -> /IO45
- J4 pad 16: unconnected-(J4-Pin_16-Pad16) -> /IO48
- J4 pad 17: unconnected-(J4-Pin_17-Pad17) -> /IO47
- U2 pad 18: (no net) -> GND
- U2 pad 19: (no net) -> GND
- U2 pad 20: (no net) -> GND
- U2 pad 21: (no net) -> GND
- U2 pad 22: (no net) -> GND
Routing:
- net /IO47: track 0.00 -> 27.9 mm, vias 0 -> 1
- net /IO48: track 0.00 -> 24.7 mm, vias 0 -> 1
- net /IO45: track 0.00 -> 21.4 mm, vias 0 -> 1
- net GND: track 1.37 -> 4.21 mm
- net /IO0: track 24.4 -> 27.0 mm
