File: esp32-pcb/esp32-pcb.kicad_sch (KiCad schematic)
At the start: 41 parts, among them J1 10118193-0001LF, J2 10118193-0001LF, J3 Conn_01x19, J4 Conn_01x19, Q1 SS8050-G, Q2 SS8050-G, U1 CP2102N-A02-GQFN28, U2 BQ24075RGTR, U3 AP2112K-3.3TRG1, X1 ESP32-S3-WROOM-1-N16R8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

Commit message: Update esp32-pcb.kicad_sch
Parts:
- added J5: Batt+, Connector_PinHeader_2.54mm:PinHeader_1x01_P2.54mm_Vertical, symbol Connector:Conn_01x01_Socket
- added J6: Batt-, Connector_PinHeader_2.54mm:PinHeader_1x01_P2.54mm_Vertical, symbol Connector:Conn_01x01_Socket
Connections:
- net GND: now also J6.1 (Pin_1)
- net VDD_BATT: now also J5.1 (Pin_1)
Other:
- moved on the sheet: D2, D3, R14, R15

Commit message: updates
Parts:
- removed J1, J2: 10118193-0001LF, 10118193-0001LF:AMPHENOL_10118193-0001LF, symbol USB-micro-receptacle:10118193-0001LF
- removed J3: Conn_01x19, Connector_PinHeader_2.54mm:PinHeader_1x19_P2.54mm_Vertical, symbol Connector_Generic:Conn_01x19
- added J1, J2: USB_B_Micro, USB-micro-receptacle:CUI_UJ2-MIBH2-4-SMT, symbol Connector:USB_B_Micro
- added J3: Conn_01x15, Connector_PinHeader_2.54mm:PinHeader_1x15_P2.54mm_Vertical, symbol Connector_Generic:Conn_01x15
- C1, C10, C11, C12, C2, C3, C4, C5, C6, C7, C8, C9: footprint Capacitor_SMD:C_01005_0402Metric_Pad0.57x0.30mm_HandSolder -> Capacitor_SMD:C_0402_1005Metric_Pad0.74x0.62mm_HandSolder
- D2, D3: footprint (none) -> Diode_SMD:D_0603_1608Metric_Pad1.05x0.95mm_HandSolder
Connections:
- net CHIP_PU: now also J3.3 (Pin_3)
- net CP_RXD: now also J4.4 (Pin_4)
- net CP_TXD: now also J4.5 (Pin_5)
- net D+: now also J2.3 (D+)
- net D-: now also J2.2 (D-)
- net GND: now also J1.5 (GND), J2.5 (GND), J3.12 (Pin_12), J3.13 (Pin_13)
- net IO0: now also J4.14 (Pin_14)
- net IO1: now also J4.2 (Pin_2)
- net IO17: now also J3.8 (Pin_8)
- net IO18: now also J3.9 (Pin_9)
- net IO2: now also J4.3 (Pin_3)
- net IO3: now also J3.11 (Pin_11)
- net IO35: now also J4.13 (Pin_13)
- net IO36: now also J4.12 (Pin_12)
- net IO37: now also J4.11 (Pin_11)
- net IO38: now also J4.10 (Pin_10)
- net IO39: now also J4.9 (Pin_9)
- net IO4: now also J3.4 (Pin_4)
- net IO40: now also J4.8 (Pin_8)
- net IO41: now also J4.7 (Pin_7)
- net IO42: now also J4.6 (Pin_6)
- net IO5: now also J3.5 (Pin_5)
- net IO6: now also J3.6 (Pin_6)
- net IO7: now also J3.7 (Pin_7)
- net IO8: now also J3.10 (Pin_10)
- net USB_D+: now also J1.3 (D+)
- net USB_D-: now also J1.2 (D-)
- net VDD_ESP: now also J4.1 (Pin_1), J3.1 (Pin_1), J3.2 (Pin_2)
- net VDD_SYS: now also J3.14 (Pin_14), J3.15 (Pin_15)
- net VDD_USB: now also J1.1 (VBUS), J2.1 (VBUS)
- no-connect marks 17 -> 15

Commit message: updates from work
Connections:
- net GND: now also U2.18, U2.19, U2.20, U2.21, U2.22
- net IO45: now also J4.15 (Pin_15)
- net IO47: now also J4.17 (Pin_17)
- net IO48: now also J4.16 (Pin_16)
Other:
- moved on the sheet: C10, C8, C9, D1, R10, R11, R12, R13, R9
